File: testbench-stm32g031-soic/testbench-stm32g031-soic.kicad_pcb (KiCad board)
At the start: 2 copper layers, 31.8 x 25.4 mm, 14 parts, among them J3 SWD, SW1 BOOT, U1 stm32g031j, U3 XC6206P362MR

Commit message: bumpdesign
Parts:
- moved C2 0.84 mm to (117.2, 55.7)
- moved J3 0.51 mm to (124.5, 58.5)
- moved SW1 0.36 mm to (124.5, 40.6)
- moved U3 0.25 mm to (120.0, 54.2)
Routing:
- net +5V: track 8.16 -> 7.32 mm
- net GND: track 86.4 -> 87.0 mm
Changed lines of the file:
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@@
     (thickness 1.6)
     (drawings 32)
-    (tracks 153)
+    (tracks 154)
     (zones 0)
     (modules 14)
@@
     (solder_mask_min_width 0.25)
     (aux_axis_origin 0 0)
-    (grid_origin 119.78 48.907499)
+    (grid_origin 111.76 38.735)
     (visible_elements FFFFFF7F)
     (pcbplotparams
@@
   )
   (module Button_Switch_SMD:SW_SPST_EVPBF (layer F.Cu)
-    (at 124.098 40.588999)
+    (at 124.46 40.588999)
     (descr "Light Touch Switch")
     (attr smd)
@@
   )
   (module Capacitor_SMD:C_0603_1608Metric (layer F.Cu)
-    (at 116.3575 55.727499 270)
+    (at 117.2 55.715 270)
     (descr "Capacitor SMD 0603 (1608 Metric), square (rectangular) end terminal, IPC_7351 nominal, (Body size source: http://www.tortai-tech.com/upload/download/2011102023233369053.pdf), generated with kicad-footprint-generator")
     (tags capacitor)
     (attr smd)
-    (fp_text reference C2 (at 0 -1.43 90) (layer F.SilkS)
+    (fp_text reference C2 (at 2.61 0.99 90) (layer F.SilkS)
       (effects (font (size 1 1) (thickness 0.15)))
     )
@@
   )
   (module cnlohr-kicad:POGO-5-SWD (layer F.Cu)
-    (at 124.46 59.055)
+    (at 124.46 58.547)
     (fp_text reference J3 (at 7.62 0) (layer F.SilkS)
       (effects (font (size 1 1) (thickness 0.15)))
     )
-    (fp_text value SWD (at -8.255 0.635) (layer F.SilkS)
+    (fp_text value SWD (at -7.87 1.548) (layer F.SilkS)
       (effects (font (size 1 1) (thickness 0.15)))
     )
@@
   )
   (module Package_TO_SOT_SMD:SOT-23 (layer F.Cu)
-    (at 120.015 53.975 270)
+    (at 120.015 54.229 270)
     (descr "SOT-23, Standard")
     (tags SOT-23)
@@
   (via (at 124.352 40.017499) (size 0.8) (drill 0.4) (layers F.Cu B.Cu) (net 1))
   (segment (start 114.7 42.811499) (end 124.352 40.017499) (width 0.25) (layer B.Cu) (net 1))
+  (segment (start 123.59 48.907499) (end 123.18 48.407499) (width 0.25) (layer F.Cu) (net 1))
   (segment (start 121.985 47.625) (end 119.38 47.319999) (width 0.25) (layer F.Cu) (net 2))
   (segment (start 119.38 47.319999) (end 116.185 46.99) (width 0.25) (layer F.Cu) (net 2))
@@
   (segment (start 118.002 52.082499) (end 118.637 51.701499) (width 0.25) (layer F.Cu) (net 5))
   (segment (start 116.185 52.07) (end 118.002 52.082499) (width 0.25) (layer F.Cu) (net 5))
-  (segment (start 116.185 52.07) (end 118.129 53.733499) (width 0.25) (layer F.Cu) (net 5))
-  (segment (start 122.447 54.749499) (end 123.971 56.019499) (width 0.25) (layer F.Cu) (net 5))
   (segment (start 123.971 56.019499) (end 124.352 56.908499) (width 0.25) (layer F.Cu) (net 5))
   (segment (start 124.352 56.908499) (end 124.46 59.055) (width 0.25) (layer F.Cu) (net 5))
-  (segment (start 121.05 54.114499) (end 122.447 54.749499) (width 0.25) (layer F.Cu) (net 5))
-  (segment (start 118.129 53.733499) (end 119.526 53.987499) (width 0.25) (layer F.Cu) (net 5))
-  (segment (start 119.526 53.987499) (end 121.05 54.114499) (width 0.25) (layer F.Cu) (net 5))
+  (segment (start 121.04 54.275) (end 122.447 54.749499) (width 0.25) (layer F.Cu) (net 5))
+  (segment (start 118.75 54.145) (end 121.04 54.275) (width 0.25) (layer F.Cu) (net 5))
+  (segment (start 122.447 54.749499) (end 123.971 56.019499) (width 0.25) (layer F.Cu) (net 5))
+  (segment (start 118.23 53.955) (end 118.75 54.145) (width 0.25) (layer F.Cu) (net 5))
+  (segment (start 116.185 52.07) (end 118.23 53.955) (width 0.25) (layer F.Cu) (net 5))
   (segment (start 111.145 44.45) (end 116.185 44.45) (width 0.25) (layer F.Cu) (net 6))
   (segment (start 116.185 44.45) (end 118.129 44.462499) (width 0.25) (layer F.Cu) (net 6))
@@
   (segment (start 132.735 52.07) (end 137.775 52.07) (width 0.25) (layer F.Cu) (net 9))
   (segment (start 120.015 54.975) (end 121.92 59.055) (width 0.25) (layer F.Cu) (net 10))
-  (segment (start 116.3575 54.939999) (end 120.015 54.975) (width 0.25) (layer F.Cu) (net 10))
+  (segment (start 117.2 54.9275) (end 120.015 54.975) (width 0.25) (layer F.Cu) (net 10))
   (zone (net 1) (net_name GND) (layer F.Cu) (hatch edge 0.508)
     (connect_pads (clearance 0.254))
